File: kicad/acsi2sd1.sch (KiCad schematic (older format))
At the start: 48 parts, among them J1 DB19_Male, J2 Jack-DC, U1 CY8C5268AXI-LP047, U6 LDO 3.3V, X2 MINI-USB-32005-201, X3 MICROSD, X4 MiniProg, X5 KitProg

Commit message: Add files via upload
Parts:
- F1B1: value MF-NSMF150-2 -> 1206L012WR
- F2B1: value MF-NSMF050-2 -> 1206L012WR
- R3, R4, R5: value 1k2 -> 1k5
- U1: value CY8C5268AXI-LP047 -> CY8C5468AXI-LP042
Changed lines of the file:
@@
 P 7850 4300
 F 0 "U1" H 7750 4350 59  0000 L BNN
-F 1 "CY8C5268AXI-LP047" H 7750 4200 59  0000 L BNN
+F 1 "CY8C5468AXI-LP042" H 7750 4200 59  0000 L BNN
 F 2 "scsi2sd12:TQFP100-14X14" H 7850 4300 50  0001 C CNN
 F 3 "" H 7850 4300 50  0001 C CNN
@@
 P 2650 2450
 F 0 "F1B1" H 2500 2509 59  0000 L BNN
-F 1 "MF-NSMF150-2" H 2100 2300 59  0000 L BNN
+F 1 "1206L012WR" H 2350 2300 59  0000 L BNN
 F 2 "scsi2sd12:R1206" H 2650 2450 50  0001 C CNN
 F 3 "" H 2650 2450 50  0001 C CNN
@@
 P 7150 8000
 F 0 "F2B1" H 7000 8059 59  0000 L BNN
-F 1 "MF-NSMF050-2" H 7000 7870 59  0000 L BNN
+F 1 "1206L012WR" H 6900 7850 59  0000 L BNN
 F 2 "scsi2sd12:R1206" H 7150 8000 50  0001 C CNN
 F 3 "" H 7150 8000 50  0001 C CNN
@@
 P 10650 2700
 F 0 "R3" H 10500 2759 59  0000 L BNN
-F 1 "1k2" H 10500 2570 59  0000 L BNN
+F 1 "1k5" H 10500 2570 59  0000 L BNN
 F 2 "scsi2sd12:R0805" H 10650 2700 50  0001 C CNN
 F 3 "" H 10650 2700 50  0001 C CNN
@@
 P 11050 2700
 F 0 "R4" H 10900 2759 59  0000 L BNN
-F 1 "1k2" H 10900 2570 59  0000 L BNN
+F 1 "1k5" H 10900 2570 59  0000 L BNN
 F 2 "scsi2sd12:R0805" H 11050 2700 50  0001 C CNN
 F 3 "" H 11050 2700 50  0001 C CNN
@@
 P 11450 2700
 F 0 "R5" H 11300 2759 59  0000 L BNN
-F 1 "1k2" H 11300 2570 59  0000 L BNN
+F 1 "1k5" H 11300 2570 59  0000 L BNN
 F 2 "scsi2sd12:R0805" H 11450 2700 50  0001 C CNN
 F 3 "" H 11450 2700 50  0001 C CNN
